File: GPIO Board Rev 3 V5.sch (EAGLE design)
At the start: 143 parts, among them J1 HEADER-2, U1 TM4C123GH6PMI, U10 SN74LVC1T45-Q1, U11 SN74LVC1T45-Q1, U12 SN74LVC1T45-Q1, U13 SN74LVC1T45-Q1, U14 SN74LVC1T45-Q1, U15 R-78E5.0-0.5, U16 ISO1050DUB, U5 SN74LVC1T45-Q1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

Commit message: V5
this should be the barebones schematic.
Connections:
- removed net SCL: D11.C, D13.C, R23.1, R24.2, R26.1
- removed net SDA: D10.C, D12.C, R24.1, R25.1
- net I2CSCL: now also D11.C, D13.C, R23.1, R24.2, R26.1
- net I2CSDA: now also D10.C, D12.C, R24.1, R25.1
Changed lines of the file:
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@@
 <label x="-83.82" y="-17.78" size="1.778" layer="95" rot="R180"/>
+</segment>
+<segment>
+<pinref part="R26" gate="G$1" pin="1"/>
+<wire x1="22.86" y1="-106.68" x2="15.24" y2="-106.68" width="0.1524" layer="91"/>
+<pinref part="D13" gate="G$1" pin="C"/>
+<wire x1="15.24" y1="-106.68" x2="5.08" y2="-106.68" width="0.1524" layer="91"/>
+<wire x1="5.08" y1="-106.68" x2="-15.24" y2="-106.68" width="0.1524" layer="91"/>
+<wire x1="-15.24" y1="-106.68" x2="-30.48" y2="-106.68" width="0.1524" layer="91"/>
+<wire x1="15.24" y1="-114.3" x2="15.24" y2="-106.68" width="0.1524" layer="91"/>
+<junction x="15.24" y="-106.68"/>
+<pinref part="D11" gate="G$1" pin="C"/>
+<wire x1="5.08" y1="-114.3" x2="5.08" y2="-106.68" width="0.1524" layer="91"/>
+<junction x="5.08" y="-106.68"/>
+<pinref part="R23" gate="G$1" pin="1"/>
+<wire x1="-15.24" y1="-99.06" x2="-15.24" y2="-106.68" width="0.1524" layer="91"/>
+<junction x="-15.24" y="-106.68"/>
+<pinref part="R24" gate="G$1" pin="2"/>
+<wire x1="-15.24" y1="-114.3" x2="-15.24" y2="-106.68" width="0.1524" layer="91"/>
+<label x="-30.48" y="-106.68" size="1.778" layer="95" rot="R180"/>
 </segment>
 </net>
@@
 <wire x1="-76.2" y1="-20.32" x2="-83.82" y2="-20.32" width="0.1524" layer="91"/>
 <label x="-83.82" y="-20.32" size="1.778" layer="95" rot="R180"/>
+</segment>
+<segment>
+<pinref part="R25" gate="G$1" pin="1"/>
+<wire x1="22.86" y1="-139.7" x2="15.24" y2="-139.7" width="0.1524" layer="91"/>
+<pinref part="R24" gate="G$1" pin="1"/>
+<wire x1="15.24" y1="-139.7" x2="5.08" y2="-139.7" width="0.1524" layer="91"/>
+<wire x1="5.08" y1="-139.7" x2="-15.24" y2="-139.7" width="0.1524" layer="91"/>
+<wire x1="-15.24" y1="-139.7" x2="-30.48" y2="-139.7" width="0.1524" layer="91"/>
+<wire x1="-15.24" y1="-124.46" x2="-15.24" y2="-139.7" width="0.1524" layer="91"/>
+<junction x="-15.24" y="-139.7"/>
+<pinref part="D12" gate="G$1" pin="C"/>
+<wire x1="15.24" y1="-144.78" x2="15.24" y2="-139.7" width="0.1524" layer="91"/>
+<junction x="15.24" y="-139.7"/>
+<pinref part="D10" gate="G$1" pin="C"/>
+<wire x1="5.08" y1="-144.78" x2="5.08" y2="-139.7" width="0.1524" layer="91"/>
+<junction x="5.08" y="-139.7"/>
+<label x="-30.48" y="-139.7" size="1.778" layer="95" rot="R180"/>
 </segment>
 </net>
@@
 </segment>
 </net>
-<net name="SCL" class="0">
-<segment>
-<pinref part="R26" gate="G$1" pin="1"/>
-<wire x1="22.86" y1="-106.68" x2="15.24" y2="-106.68" width="0.1524" layer="91"/>
-<pinref part="D13" gate="G$1" pin="C"/>
-<wire x1="15.24" y1="-106.68" x2="5.08" y2="-106.68" width="0.1524" layer="91"/>
-<wire x1="5.08" y1="-106.68" x2="-15.24" y2="-106.68" width="0.1524" layer="91"/>
-<wire x1="-15.24" y1="-106.68" x2="-30.48" y2="-106.68" width="0.1524" layer="91"/>
-<wire x1="15.24" y1="-114.3" x2="15.24" y2="-106.68" width="0.1524" layer="91"/>
-<junction x="15.24" y="-106.68"/>
-<pinref part="D11" gate="G$1" pin="C"/>
-<wire x1="5.08" y1="-114.3" x2="5.08" y2="-106.68" width="0.1524" layer="91"/>
-<junction x="5.08" y="-106.68"/>
-<pinref part="R23" gate="G$1" pin="1"/>
-<wire x1="-15.24" y1="-99.06" x2="-15.24" y2="-106.68" width="0.1524" layer="91"/>
-<junction x="-15.24" y="-106.68"/>
-<pinref part="R24" gate="G$1" pin="2"/>
-<wire x1="-15.24" y1="-114.3" x2="-15.24" y2="-106.68" width="0.1524" layer="91"/>
-<label x="-30.48" y="-106.68" size="1.778" layer="95" rot="R180"/>
-</segment>
-</net>
-<net name="SDA" class="0">
-<segment>
-<pinref part="R25" gate="G$1" pin="1"/>
-<wire x1="22.86" y1="-139.7" x2="15.24" y2="-139.7" width="0.1524" layer="91"/>
-<pinref part="R24" gate="G$1" pin="1"/>
-<wire x1="15.24" y1="-139.7" x2="5.08" y2="-139.7" width="0.1524" layer="91"/>
-<wire x1="5.08" y1="-139.7" x2="-15.24" y2="-139.7" width="0.1524" layer="91"/>
-<wire x1="-15.24" y1="-139.7" x2="-30.48" y2="-139.7" width="0.1524" layer="91"/>
-<wire x1="-15.24" y1="-124.46" x2="-15.24" y2="-139.7" width="0.1524" layer="91"/>
-<junction x="-15.24" y="-139.7"/>
-<pinref part="D12" gate="G$1" pin="C"/>
-<wire x1="15.24" y1="-144.78" x2="15.24" y2="-139.7" width="0.1524" layer="91"/>
-<junction x="15.24" y="-139.7"/>
-<pinref part="D10" gate="G$1" pin="C"/>
-<wire x1="5.08" y1="-144.78" x2="5.08" y2="-139.7" width="0.1524" layer="91"/>
-<junction x="5.08" y="-139.7"/>
-<label x="-30.48" y="-139.7" size="1.778" layer="95" rot="R180"/>
-</segment>
-</net>
