File: GPIO Board Rev 3 V5.sch (EAGLE design)
At the start: 139 parts, among them J1 HEADER-2, U1 TM4C123GH6PMI, U10 SN74LVC1T45-Q1, U11 SN74LVC1T45-Q1, U12 SN74LVC1T45-Q1, U13 SN74LVC1T45-Q1, U14 SN74LVC1T45-Q1, U15 R-78E5.0-0.5, U16 ISO1050DUB, U5 SN74LVC1T45-Q1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

Commit message: 1
Parts:
- removed X9: MICRO-FIT_3.0_6POS_2ROW_R/A, gtsr-connector:MICRO-FIT_3.0_6POS_2ROW_R/A
- added X5, X6: MICRO-FIT_3.0_6POS_2ROW, gtsr-connector:MICRO-FIT_3.0_6POS_2ROW
Connections:
- new net +12V: CAN3.1, CAN3.3, CAN3.5, CAN4.1, CAN4.3, CAN4.5, U15.+VIN
- new net 5V: X6.5
- new net GNDCAN: C38.2, CAN3.2, CAN3.4, CAN3.6, CAN4.2, CAN4.4, CAN4.6
- new net GPIOEXT0: U1.47-PB2/I2C0SCL/T3CCP0, X5.1
- new net GPIOEXT1: U1.48-PB3/I2C0SDA/T3CCP1, X5.2
- new net GPIOEXT2: U1.4-PB7/M0PWM1/SSI2TX/T0CCP1, X5.3
- new net GPIOEXT3: U1.5-PF4/IDX0/M1FAULT0/T2CCP0/USB0EPEN, X5.4
- new net GPIOEXT4: U1.13-PC7/CO-/U3TX/USB0PFLT/WT1CCP1, X5.5
- new net GPIOEXT5: U1.14-PC6/C0+/PHB1/U3RX/USB0EPEN/WT1CCP0, X5.6
- new net VOUT1: C8.1, R4.1, TP1.1
- new net VOUT2: C10.1, R8.1, TP2.1
- new net VOUT3: C12.1, R12.1, TP3.1
- new net VOUT4: C14.1, R31.1, TP15.1
- net +3V3: now also X6.6; no longer X9.6
- net +5V: no longer X9.5
- net +VIN: no longer CAN3.1, CAN3.3, CAN3.5, CAN4.1, CAN4.3, CAN4.5, U15.+VIN
- net -VIN: no longer C38.2, CAN3.2, CAN3.4, CAN3.6, CAN4.2, CAN4.4, CAN4.6
- net GND: now also X6.2, X6.3; no longer X9.2, X9.3
- net N$51: now also X6.4; no longer X9.4
- net N$52: now also X6.1; no longer X9.1
- net TIVAA1: no longer C8.1, R4.1, TP1.1
- net TIVAA2: no longer C10.1, R8.1, TP2.1
- net TIVAA3: no longer C12.1, R12.1, TP3.1
- net TIVAA4: no longer C14.1, R31.1, TP15.1
