File: GPIO Board Rev 3 V5.brd (EAGLE design)
At the start: 104.1 x 77.7 mm, 140 parts, among them J1 HEADER-2, U1 TM4C123GH6PMI, U10 SN74LVC1T45-Q1, U11 SN74LVC1T45-Q1, U12 SN74LVC1T45-Q1, U13 SN74LVC1T45-Q1, U14 SN74LVC1T45-Q1, U15 R-78E5.0-0.5, U16 ISO1050DUB, U5 SN74LVC1T45-Q1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

Commit message: 1
1
Parts:
- moved C19 190.2 mm to (90.2, 68.8)
- moved R17 185.5 mm to (105.3, 65.4)
- moved R18 185.4 mm to (98.8, 65.5)
- moved TP5 183.4 mm to (89.9, 65.8)
- moved U9 171.6 mm to (105.7, 67.8), turned to 270 degrees
- moved C36 170.0 mm to (69.1, 68.1)
- moved U10 169.8 mm to (98.8, 67.8), turned to 270 degrees
- moved C35 164.8 mm to (69.1, 69.1)
- moved U14 162.7 mm to (71.4, 68.1), turned to 270 degrees
- moved C28 157.0 mm to (96.5, 68.1)
- moved C6 156.3 mm to (60.7, 8.13)
- moved D1 155.6 mm to (71.9, 41.7), turned to 180 degrees
- moved R27 155.6 mm to (81.0, 18.8)
- moved R14 154.2 mm to (93.0, 65.0)
- moved C34 153.8 mm to (62.7, 68.1)
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Routing:
- net RESET: track 0.00 -> 137.7 mm, vias 0 -> 4
- net VCC: track 0.00 -> 129.2 mm, vias 0 -> 3
- net +3V3: track 0.00 -> 100.7 mm, vias 0 -> 2
- net +12V: track 0.00 -> 86.5 mm, vias 0 -> 2
- net TIVAD8: track 0.00 -> 77.1 mm, vias 0 -> 2
- net TIVAD5: track 0.00 -> 72.9 mm, vias 0 -> 4
- net TIVAD9: track 0.00 -> 72.4 mm, vias 0 -> 4
- net TIVAD6: track 0.00 -> 69.9 mm, vias 0 -> 4
- net TIVADIR6: track 0.00 -> 67.7 mm, vias 0 -> 4
- net CANTX: track 0.00 -> 67.5 mm, vias 0 -> 4
- net TIVAD10: track 0.00 -> 66.2 mm, vias 0 -> 4
- net TIVADIR5: track 0.00 -> 65.3 mm, vias 0 -> 2
- net N$6: track 0.00 -> 63.6 mm, vias 0 -> 1
- net TMS: track 0.00 -> 61.0 mm, vias 0 -> 6
- net TIVADIR10: track 0.00 -> 60.2 mm, vias 0 -> 4
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
Commit message: 1
1
Routing:
- net GND: track 15.1 -> 150.0 mm, vias 0 -> 15
- net UARTTX: track 3.57 -> 79.6 mm, vias 1 -> 6
- net VCC: track 129.2 -> 189.8 mm, vias 3 -> 13
- net UARTRX: track 4.58 -> 56.8 mm, vias 1 -> 5
- net +3V3: track 100.7 -> 139.3 mm, vias 2 -> 4
- net GPIOEXT5: track 47.0 -> 53.8 mm
- net GPIOEXT4: track 45.7 -> 47.4 mm
- added copper zone on layer 16, net GND
- added copper zone on layer 1, net VCC

Commit message: 1
1
Parts:
- added A1: SR3-MED-WITH-TEXT, gtsr-aesthetic:SR3_MED
- added _LOG1: LOGO-LG, gtsr-aesthetic:GTSR_LOGO_LG
Changed lines of the file:
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@@
 <attribute name="SUPPLIER_PN" value="WM1791-ND" x="15.494" y="72.136" size="1.778" layer="27" display="off"/>
 </element>
+<element name="_LOG1" library="gtsr-aesthetic" package="GTSR_LOGO_LG" value="LOGO-LG" x="5.08" y="2.032" smashed="yes"/>
+<element name="A1" library="gtsr-aesthetic" package="SR3_MED" value="SR3-MED-WITH-TEXT" x="100.838" y="5.08" smashed="yes"/>
 </elements>
 <signals>
